File: LINEAR POWER SUPPLY/LINEAR POWER SUPPLY.kicad_pcb (KiCad board)
At the start: 2 copper layers, 8 parts, among them J1 Conn_01x01_Pin, J2 Conn_01x01_Pin, J3 Conn_01x01_Pin

Commit message: sdfasf
Parts:
- added BR1: GBJ2510-F, PCB:GBJ_1, F.Cu at (49.7, 81.9)
- added Q1: 2SB817, Package_TO_SOT_THT:TO-3PB-3_Vertical, F.Cu at (52.1, 91.2)
- added R1: R, Resistor_THT:R_Axial_DIN0516_L15.5mm_D5.0mm_P7.62mm_Vertical, F.Cu at (69.4, 91.4)
- added TH1: Thermistor_NTC, Resistor_THT:R_Axial_Power_L38.0mm_W6.4mm_P40.64mm, F.Cu at (50.9, 77.2)
- D1: value GBJ2510-F -> D_Zener_Filled; footprint PCB:GBJ_1 -> Diode_THT:D_DO-15_P5.08mm_Vertical_KathodeUp
- J1, J2, J3: value Conn_01x01_Pin -> SPADE
- moved D1 6.95 mm to (63.9, 56.0)
Connections:
- D1 pad 1: +DC -> Net-(D1-K)
- D1 pad 2: Net-(J2-Pin_1) -> unconnected-(D1-A-Pad2)
