File: LINEAR POWER SUPPLY/LINEAR POWER SUPPLY.kicad_pcb (KiCad board)
At the start: 2 copper layers, 12 parts, among them J1 SPADE, J2 SPADE, J3 SPADE, Q1 2SB817

Commit message: 26-07-2026
Parts:
- added F1: Fuse_Small, Fuse:Fuseholder_Cylinder-5x20mm_Stelvio-Kontek_PTF78_Horizontal_Open, F.Cu at (131.9, 45.9)
- added U1: LM317_TO-220, Package_TO_SOT_THT:TO-220-3_Vertical, F.Cu at (132.8, 55.3)
- added U2: ACS712xLCTR-05B, Package_SO:SOIC-8_3.9x4.9mm_P1.27mm, F.Cu at (145.3, 54.7)
Connections:
- BR1 pad 1: unconnected-(BR1-+-Pad1) -> Net-(BR1-+)
- D1 pad 2: unconnected-(D1-A-Pad2) -> Net-(D1-A)
- Q1 pad 3: unconnected-(Q1-E-Pad3) -> Net-(D3-K)
- TH1 pad 1: unconnected-(TH1-Pad1) -> Net-(F1-Pad2)
- TH1 pad 2: unconnected-(TH1-Pad2) -> +DC
