File: SOLDERING IRON/SOLDERING IRON.kicad_sch (KiCad schematic)
At the start: 53 parts, among them J1 Conn_01x02, J2 Conn_01x02, J3 Conn_01x02, SW1 SW_DIP_x01, SW2 SW_DIP_x01, U1 ESP32-WROOM-32U, U2 NE555D, U3 Opamp_Dual, U4 Opamp_Dual, U5 LM2576HVS-3.3, U6 PEC11H-4215F-S0024

Commit message: 26-07-2026
Parts:
- removed C10: 0.1UF, Capacitor_THT:C_Disc_D8.0mm_W5.0mm_P10.00mm, symbol Device:C
- removed MOSFET1: NTBLS0D7N06C, H-PSOF8L_100CU_ONS, symbol RUPESH:NTBLS0D7N06C
- removed R24, R25: 1K, PCB:1_4W RES, symbol Device:R
- removed R4: 120E, PCB:1_4W RES, symbol Device:R
- removed U2: NE555D, Package_DIP:DIP-8_W7.62mm_LongPads, symbol Timer:NE555D
- added C10, C11: 1000uf, Capacitor_SMD:C_1206_3216Metric_Pad1.33x1.80mm_HandSolder, symbol Device:C_Polarized
- added D5, D6, D7: 1N4148, Diode_SMD:D_SMC_Handsoldering, symbol dk_Diodes-Rectifiers-Single:1N4148
- added Q1: BC846, Package_TO_SOT_SMD:SOT-23_Handsoldering, symbol Transistor_BJT:BC846
- added Q2: NTBLS1D5N10MCTXG, PCB:NVBLS0D8N08XTXG, symbol SamacSys_Parts:NTBLS1D5N10MCTXG
- added Q3: BC856, Package_TO_SOT_SMD:SOT-23_Handsoldering, symbol Transistor_BJT:BC856
- added R10: 120E, Resistor_SMD:R_1206_3216Metric_Pad1.30x1.75mm_HandSolder, symbol Device:R
- added U7: L7805, Package_TO_SOT_THT:TO-220-3_Horizontal_TabDown, symbol Regulator_Linear:L7805
- C1, C2, C3, C6, C7, C9: value 0.1UF -> C; footprint Capacitor_THT:C_Disc_D8.0mm_W5.0mm_P10.00mm -> Capacitor_SMD:C_1206_3216Metric_Pad1.33x1.80mm_HandSolder
- C4, C8: footprint Capacitor_THT:CP_Radial_D12.5mm_P7.50mm -> Capacitor_SMD:C_1206_3216Metric_Pad1.33x1.80mm_HandSolder
- C5: footprint Capacitor_THT:CP_Radial_D10.0mm_P5.00mm -> Capacitor_SMD:C_1206_3216Metric_Pad1.33x1.80mm_HandSolder
- D1, D2, D3, D4: footprint Diode_THT:D_A-405_P7.62mm_Horizontal -> Diode_SMD:D_SMC_Handsoldering
- R1, R11, R12, R13, R14, R3, R5, R7, R8, R9: footprint PCB:1_4W RES -> Resistor_SMD:R_1206_3216Metric_Pad1.30x1.75mm_HandSolder
- R15, R16, R17, R18, R19, R20, R21, R22, R6: value 0E -> 0E01; footprint PCB:1_4W RES -> Resistor_SMD:R_1206_3216Metric_Pad1.30x1.75mm_HandSolder
- R2: value 0E -> 0e; footprint PCB:1_4W RES -> Resistor_SMD:R_1206_3216Metric_Pad1.30x1.75mm_HandSolder
- R23: value 4K7 -> 1K; footprint PCB:1_4W RES -> Resistor_SMD:R_1206_3216Metric_Pad1.30x1.75mm_HandSolder
- SW1, SW2: footprint PCB:SW_PUSH_6mm_H7.3mm_THT -> Button_Switch_THT:SW_PUSH_6mm_H7.3mm
- U6: footprint PEC11H4215FS0024 -> PCB:PEC11H4215FS0024
Connections:
- net R/W is gone; now on net GND: R21.1
- net +12V: now also Q1.3 (C); no longer DS1.4 (VDD), R13.1, RV1.3
- net CURRENT: now also R8.1, U3.7
- net DRAIN: now also Q2.10 (D_2), Q2.11 (D_3), Q2.12 (D_4), Q2.9 (D_1)
- net GND: now also R23.2, U4.6 (-), C10.2, C11.2, D7.2, Q3.2 (E), R10.2, U7.2 (GND); no longer R23.1
- net IR: now also Q2.2 (S_1), Q2.3 (S_2), Q2.4 (S_3), Q2.5 (S_4), Q2.6 (S_5), Q2.7 (S_6), Q2.8 (S_7)
- net LINE: now also D5.2
- net TEMPETURE: now also U4.7
- net at U3.1, U3.2 (-), U3.5 (+): now also R10.1
- net at R5.1: now also Q1.1 (B), Q3.1 (B)
- new net: C10.1, D5.1, D6.1, U7.1 (IN)
- new net: Q1.2 (E), Q2.1 (G), Q3.3 (C)
- new net +5V: C11.1, D6.2, D7.1, DS1.4 (VDD), R13.1, R23.1, RV1.3, U7.3 (OUT)
